File: kicad/Hearth.kicad_sch (KiCad schematic)
At the start: 0 parts

Commit message: Modifiyng Schema
Parts:
- added BT1: 800mAh, symbol EUB_Mechanical:MECH_BATTERY_CELL_1S_EUB
- added C1, C10, C11, C14, C15, C17, C18, C3, C4, C7, C8: 22μ, symbol Device:C_Small
- added C12, C13, C16, C2, C5, C9: 100n, symbol Device:C_Small
- added C6: 10μ, symbol Device:C_Small
- added D1: LED_EXT, symbol Device:LED
- added D2: LED_CHG, symbol Device:LED
- added D3: LED_FULL/PGOOD, symbol Device:LED
- added D4: ESD9B5.0ST5G, Diode_SMD:D_SOD-923, symbol Diode:ESD9B5.0ST5G
- added F1: Polyfuse, symbol Device:Polyfuse
- added FB1: FerriteBead_Small, symbol Device:FerriteBead_Small
- added J1: USB_C_Receptacle_USB2.0_16P, EUB_Connector:USB_C_Receptacle_G-Switch_GT-USB-7010ASV_NOSILK, symbol Connector:USB_C_Receptacle_USB2.0_16P
- added J2: Conn_01x02_Pin, symbol Connector:Conn_01x02_Pin
- added J3: Barrel_Jack_Switch_Pin3Ring, symbol Connector:Barrel_Jack_Switch_Pin3Ring
- added J4: EUB_BUS, symbol Connector:Conn_01x05_Pin
- added L1: 4.7μ, symbol Device:L
- added R1, R2, R6, R7, R8: 5.1k, EUB_Passive:R_0603_1608Metric_NOSILK_EUB, symbol Device:R_US
- added R3, R4, R5: 1k, EUB_Passive:R_0603_1608Metric_NOSILK_EUB, symbol Device:R_US
- added TH1: Thermistor, symbol Device:Thermistor
- added TP1: TP_USB5V, TestPoint:TestPoint_Pad_2.0x2.0mm, symbol Connector:TestPoint
- added TP2: TP_CHG, TestPoint:TestPoint_Pad_2.0x2.0mm, symbol Connector:TestPoint
- added TP3: TP_PGOOD, TestPoint:TestPoint_Pad_2.0x2.0mm, symbol Connector:TestPoint
- added TP4: TP_DC9V, TestPoint:TestPoint_Pad_2.0x2.0mm, symbol Connector:TestPoint
- added TP5: TP_DC5V, TestPoint:TestPoint_Pad_2.0x2.0mm, symbol Connector:TestPoint
- added TP6: TP_BQ_SYS, TestPoint:TestPoint_Pad_2.0x2.0mm, symbol Connector:TestPoint
- added TP7: TP_3V3, TestPoint:TestPoint_Pad_2.0x2.0mm, symbol Connector:TestPoint
- added TP8: TP_SYS_5V, TestPoint:TestPoint_Pad_2.0x2.0mm, symbol Connector:TestPoint
- added TP9: TP_GND, TestPoint:TestPoint_Pad_2.0x2.0mm, symbol Connector:TestPoint
- added U1: TPS61023DRLR_EUB, Package_TO_SOT_SMD:SOT-563, symbol EUB_Power:TPS61023DRLR_EUB
- added U2: BQ24074RGT, Package_DFN_QFN:VQFN-16-1EP_3x3mm_P0.5mm_EP1.6x1.6mm, symbol Battery_Management:BQ24074RGT
- added U3: LM5050-1, Package_TO_SOT_SMD:TSOT-23-6, symbol Power_Management:LM5050-1
- added U4: MP2338, Package_TO_SOT_SMD:SOT-583-8, symbol EUB_Power:MP2338
- added U5: AP7333-33SAG-7, EUB_Package:SOT-23-3_NOSILK, symbol EUB_Power:AP7333-33SAG-7
- added U6: TPS2121, symbol Power_Management:TPS2412D
Connections:
- new net: C6.2, J2.1 (Pin_1), U2.2 (BAT), U2.3 (BAT)
- new net: D2.2 (A), R4.2
- new net: TH1.1, U2.1 (TS)
- new net: R8.2, U2.15 (ITERM)
- new net: U2.17 (VSS), U2.8 (VSS)
- new net: TP2.1, U2.7 (~{PGOOD})
- new net: TP3.1, U2.9 (~{CHG})
- new net: D1.2 (A), R3.2
- new net: F1.1, J1.A4 (VBUS), J1.A9 (VBUS), J1.B4 (VBUS), J1.B9 (VBUS), TP1.1
- new net: R6.1, R7.2, U1.1 (FB)
- new net: D3.2 (A), R5.2
- new net: L1.2, U1.5 (SW)
- new net: J1.A5 (CC1), R1.1
- new net: J1.B5 (CC2), R2.1
- new net 3V3: C13.2, C14.2, C15.2, J4.2 (+3V3), TP7.1, U5.2 (VO)
- new net BOOST5V: C10.2, C11.2, C12.2, R6.2, U1.6 (VOUT), U6.2 (IN2)
- new net BQ_SYS: C3.2, C4.2, C5.2, C7.2, C8.2, C9.2, L1.1, TP6.1, U1.2 (EN), U1.3 (VIN), U2.10 (OUT), U2.11 (OUT)
- new net BQ_VIN: C1.2, C2.2, FB1.2, U2.13 (IN)
- new net DC5V: TP5.1, U6.7 (IN1)
- new net DC9V_IN: J3.3, TP4.1, U4.2 (IN)
- new net EUB_CHG: J4.4 (CHG_N)
- new net EUB_PGOOD: J4.3 (PGOOD_N)
- new net GND: C1.1, C10.1, C11.1, C12.1, C13.1, C14.1, C15.1, C16.1, C17.1, C18.1, C2.1, C3.1, C4.1, C5.1, C6.1, C7.1, C8.1, C9.1, D4.2 (A2), J1.A1 (GND), J1.A12 (GND), J1.B1 (GND), J1.B12 (GND), J1.S1 (SHIELD), J2.2 (Pin_2), J3.1, J4.5 (GND), R1.2, R2.2, R7.1, TH1.2, TP9.1, U1.4 (GND), U2.14 (TMR), U2.4 (~{CE}), U4.4 (GND), U5.3 (GND), U6.12 (GND)
- new net SYS_5V: C16.2, C17.2, C18.2, J4.1 (+5V), TP8.1, U5.1 (VI), U6.8 (OUT)
- new net USB5V_IN: D4.1 (A1), F1.2, FB1.1
- no-connect marks 0 -> 6
Other:
- note added: "Block A：USB入力（5V）＋ESD"
- note added: "Block B：充電＋PowerPath（USB → LiPo / SYS生成）"
- note added: "Block C：バッテリー/PowerPathレール → 5V昇圧（BOOST5V）"
- note added: "Block D：DC9V入力（センターマイナス）＋理想ダイオード逆接保護"
- note added: "Block E：DC9V → 5V降圧（DC5V）"
- note added: "Block F：5V合流（DC優先のPower Mux）→ SYS_5V生成"
- note added: "Block G：5V → 3.3V（ロジック）"
- note added: "Block H：PGOOD/CHG（状態通知）とEUB-BUSへの公開（OD）"
